File: gbfs_display/gbfs_display.kicad_pcb (KiCad board)
At the start: 2 copper layers, 69.8 x 63.5 mm, 7 parts, among them P1 power, P2 power, U1 esp8266_thing_dev

Commit message: Update PCB (I don't know what changed)
Committing this because it was saved - I honestly don't know what was
changed about it.
Parts:
- R1: footprint Resistors_ThroughHole:R_Axial_DIN0204_L3.6mm_D1.6mm_P5.08mm_Horizontal -> Resistors_ThroughHole:R_Axial_DIN0204_L3.6mm_D1.6mm_P7.62mm_Horizontal
- moved LLC1 1.42 mm to (164.1, 105.5)
- moved R1 0.38 mm to (174.9, 105.5)
- moved U1 0.06 mm to (177.9, 97.9)
Routing:
- net /GND: track 180.0 -> 257.1 mm
- net /5v: track 151.8 -> 227.6 mm
- net Net-(LLC1-PadL3): track 12.7 -> 14.1 mm
- net Net-(LLC1-PadR1): track 9.64 -> 10.9 mm
- net Net-(LLC1-PadL1): track 3.92 -> 3.22 mm
